Commit message: support for arm simulation and feedback visualization

File: robots/youbot-sensors.urdf.xacro (robot description, xacro)
@@ -28,22 +28,51 @@
        the origin block defines where the component is w.r.t its parent (in this case the parent
        is the world frame). For more, see http://www.ros.org/wiki/xacro -->
-<!-- foot for arm-->
+  <!-- foot for arm-->
   <xacro:youbot_base name="base"/>
-  <!--<xacro:youbot_plate name="plate" parent="base_link">
+  <xacro:youbot_plate name="plate" parent="base_link">
     <origin xyz="-0.159 0 0.046" rpy="0 0 0" />
-  </xacro:youbot_plate>-->
+  </xacro:youbot_plate>
   <xacro:youbot_arm name="arm" parent="base_link">
-    <!--<origin xyz="0.143 0 0.046" rpy="0 0 0" />-->
-    <origin xyz="0.123 0 0.046" rpy="0 0 0" /> <!-- x offset needs to be further verified -->
+    <origin xyz="0.143 0 0.046" rpy="0 0 0" />
   </xacro:youbot_arm>
   <xacro:youbot_gripper name="gripper" parent="arm_link_5">
     <origin xyz="0 0 0" rpy="0 0 0" />
   </xacro:youbot_gripper>
-  <xacro:youbot_arm name="arm_2" parent="base_link">
-    <!--<origin xyz="-0.143 0 0.046" rpy="0 0 3.1415" />-->
-    <origin xyz="-0.123 0 0.046" rpy="0 0 3.1415" />  <!-- x offset needs to be further verified -->
-  </xacro:youbot_arm>
-  <xacro:youbot_gripper name="gripper_2" parent="arm_2_link_5">
-    <origin xyz="0 0 0" rpy="0 0 0" />
-  </xacro:youbot_gripper>
+  <!-- BRSU SPECIFIC STUFF -->
+  <xacro:include filename="$(find youbot_description)/urdf/updated_materials.urdf.xacro" />
+  <xacro:include filename="$(find youbot_description)/urdf/misc/sensor_angle.urdf.xacro" />
+  <xacro:include filename="$(find youbot_description)/urdf/misc/cam3d_tower.urdf.xacro" />
+  <xacro:include filename="$(find youbot_description)/urdf/sensors/kinect_camera.urdf.xacro" />
+  <xacro:include filename="$(find youbot_description)/urdf/sensors/microsoft_lifecam.urdf.xacro" />
+  <xacro:include filename="$(find youbot_description)/urdf/sensors/asus_xtion_camera.urdf.xacro" />
+  <!-- base laser rear -->
+  <xacro:hokuyo_urg04_laser name="base_laser_rear" parent="base" ros_topic="scan_rear" update_rate="10" min_angle="-1.57" max_angle="1.57">
+     <origin xyz="-0.3 0.0 -0.03" rpy="0 0 ${M_PI}" />
+  </xacro:hokuyo_urg04_laser>
+  <!-- Sensor angle on arm -->
+  <xacro:sensor_angle name="arm_sensor_angle" parent="arm_link_5">
+    <origin xyz="-0.002 0.0 -0.023" rpy="0.0 0.0 0.0" />
+  </xacro:sensor_angle>
+  <!-- ASUS Xtion on arm sensor angle -->
+<!--
+  <xacro:asus_xtion_camera name="openni" parent="arm_sensor_angle_part2_link"  tilt="0.0">
+    <origin xyz="0.01 0.0 0.0" rpy="${M_PI} 0.0 ${M_PI}" />
+  </xacro:asus_xtion_camera>
+-->
+  <!-- tower -->
+<!--
+  <xacro:cam3d_tower name="tower" parent="plate_link">
+    <origin xyz="-0.0659 0.0 0.025" rpy="0 0 0" />
+  </xacro:cam3d_tower>
+-->
+  <!-- 3D camera on tower -->
+<!--
+  <xacro:kinect_camera name="openni" parent="tower_link">
+    <origin xyz="0.0509 -0.03 0.49" rpy="0 0.545 0" />
+  </xacro:kinect_camera>
+-->
+  <!-- Microsoft LifeCam on gripper -->
+  <xacro:microsoft_lifecam name="microsoft_lifecam" parent="arm_sensor_angle_part2_link">
+    <origin xyz="-0.04 0 -0.03" rpy="0 ${M_PI} 0" />
+  </xacro:microsoft_lifecam>
 </robot>

File: robots/youbot_arm.urdf.xacro (robot description, xacro)
@@ -3,21 +3,17 @@
        xmlns:controller="http://playerstage.sourceforge.net/gazebo/xmlschema/#controller"
        xmlns:interface="http://playerstage.sourceforge.net/gazebo/xmlschema/#interface"
-       xmlns:xacro="http://www.ros.org/wiki/xacro"
+       xmlns:xacro="http://playerstage.sourceforge.net/gazebo/xmlschema/#interface"
        name="youbot" >
   <!-- The following included files set up definitions of parts of the robot body -->
   <!-- misc common stuff? -->
-  <xacro:include filename="$(find youbot_description)/urdf/common.xacro"/>
-  <!-- youbot base -->
-  <xacro:include filename="$(find youbot_description)/urdf/youbot_base/base.urdf.xacro" />
-  <!-- youbot plate -->
-  <xacro:include filename="$(find youbot_description)/urdf/youbot_plate/plate.urdf.xacro" />
+  <xacro:include filename="$(find youbot_description)/urdf/common.xacro" />
+  <!-- materials for visualization -->
+  <xacro:include filename="$(find youbot_description)/urdf/materials.urdf.xacro" />
   <!-- youbot arm -->
-  <xacro:include filename="$(find youbot_description)/urdf/youbot_arm/arm.urdf.xacro"/>
-  <!-- youbot gripper -->
+  <xacro:include filename="$(find youbot_description)/urdf/youbot_arm/arm.urdf.xacro" />
+  <!-- youbot arm -->
   <xacro:include filename="$(find youbot_description)/urdf/youbot_gripper/gripper.urdf.xacro" />
   <!-- generic simulator_gazebo plugins for starting mechanism control, ros time, ros battery -->
-  <!--include filename="$(find youbot_description)/gazebo/gazebo.urdf.xacro" -->
-  <!-- materials for visualization -->
-  <xacro:include filename="$(find youbot_description)/urdf/materials.urdf.xacro" />
+  <xacro:include filename="$(find youbot_description)/gazebo/gazebo.urdf.xacro" />
   <!-- Now we can start using the macros included above to define the actual youbot -->
   <!-- The first use of a macro.  This one was defined in base.urdf.xacro above.
@@ -29,10 +25,13 @@
        is the world frame). For more, see http://www.ros.org/wiki/xacro -->
 <!-- foot for arm-->
-  <xacro:youbot_base name="base" />
-  <xacro:youbot_plate name="plate" parent="base_link">
-    <origin xyz="-0.159 0 0.046" rpy="0 0 0" />
-  </xacro:youbot_plate>
+  <link name="base_link">
+    <inertial>
+		   <origin xyz="0 0 0" rpy="0 0 0"/>
+		   <mass value="10.0"/>
+		   <inertia ixx="0.1"  ixy="0"  ixz="0" iyy="0.1" iyz="0" izz="0.1" />
+    </inertial>
+    </link>
   <xacro:youbot_arm name="arm" parent="base_link">
-    <origin xyz="0.143 0 0.046" rpy="0 0 0" />
+    <origin xyz="0 0 0" rpy="0 0 0" />
   </xacro:youbot_arm>
   <xacro:youbot_gripper name="gripper" parent="arm_link_5">

File: robots/youbot_base.urdf.xacro (robot description, xacro)
@@ -3,19 +3,13 @@
        xmlns:controller="http://playerstage.sourceforge.net/gazebo/xmlschema/#controller"
        xmlns:interface="http://playerstage.sourceforge.net/gazebo/xmlschema/#interface"
-       xmlns:xacro="http://www.ros.org/wiki/xacro"
+       xmlns:xacro="http://playerstage.sourceforge.net/gazebo/xmlschema/#interface"
        name="youbot" >
   <!-- The following included files set up definitions of parts of the robot body -->
   <!-- misc common stuff? -->
-  <xacro:include filename="$(find youbot_description)/urdf/common.xacro"/>
+  <xacro:include filename="$(find youbot_description)/urdf/common.xacro" />
   <!-- youbot base -->
   <xacro:include filename="$(find youbot_description)/urdf/youbot_base/base.urdf.xacro" />
-  <!-- youbot plate -->
-  <xacro:include filename="$(find youbot_description)/urdf/youbot_plate/plate.urdf.xacro" />
-  <!-- youbot arm -->
-  <xacro:include filename="$(find youbot_description)/urdf/youbot_arm/arm.urdf.xacro"/>
-  <!-- youbot gripper -->
-  <xacro:include filename="$(find youbot_description)/urdf/youbot_gripper/gripper.urdf.xacro" />
   <!-- generic simulator_gazebo plugins for starting mechanism control, ros time, ros battery -->
-  <!--include filename="$(find youbot_description)/gazebo/gazebo.urdf.xacro" -->
+  <xacro:include filename="$(find youbot_description)/gazebo/gazebo.urdf.xacro" />
   <!-- materials for visualization -->
   <xacro:include filename="$(find youbot_description)/urdf/materials.urdf.xacro" />
@@ -28,14 +22,4 @@
        the origin block defines where the component is w.r.t its parent (in this case the parent
        is the world frame). For more, see http://www.ros.org/wiki/xacro -->
-<!-- foot for arm-->
-  <xacro:youbot_base name="base" />
-  <xacro:youbot_plate name="plate" parent="base_link">
-    <origin xyz="-0.159 0 0.046" rpy="0 0 0" />
-  </xacro:youbot_plate>
-  <xacro:youbot_arm name="arm" parent="base_link">
-    <origin xyz="0.143 0 0.046" rpy="0 0 0" />
-  </xacro:youbot_arm>
-  <xacro:youbot_gripper name="gripper" parent="arm_link_5">
-    <origin xyz="0 0 0" rpy="0 0 0" />
-  </xacro:youbot_gripper>
+  <xacro:youbot_base name="base"/>
 </robot>

File: robots/youbot_gripper.urdf.xacro (robot description, xacro)
@@ -3,19 +3,13 @@
        xmlns:controller="http://playerstage.sourceforge.net/gazebo/xmlschema/#controller"
        xmlns:interface="http://playerstage.sourceforge.net/gazebo/xmlschema/#interface"
-       xmlns:xacro="http://www.ros.org/wiki/xacro"
+       xmlns:xacro="http://playerstage.sourceforge.net/gazebo/xmlschema/#interface"
        name="youbot" >
   <!-- The following included files set up definitions of parts of the robot body -->
   <!-- misc common stuff? -->
-  <xacro:include filename="$(find youbot_description)/urdf/common.xacro"/>
-  <!-- youbot base -->
-  <xacro:include filename="$(find youbot_description)/urdf/youbot_base/base.urdf.xacro" />
-  <!-- youbot plate -->
-  <xacro:include filename="$(find youbot_description)/urdf/youbot_plate/plate.urdf.xacro" />
-  <!-- youbot arm -->
-  <xacro:include filename="$(find youbot_description)/urdf/youbot_arm/arm.urdf.xacro"/>
+  <xacro:include filename="$(find youbot_description)/urdf/common.xacro" />
   <!-- youbot gripper -->
   <xacro:include filename="$(find youbot_description)/urdf/youbot_gripper/gripper.urdf.xacro" />
   <!-- generic simulator_gazebo plugins for starting mechanism control, ros time, ros battery -->
-  <!--include filename="$(find youbot_description)/gazebo/gazebo.urdf.xacro" -->
+  <xacro:include filename="$(find youbot_description)/gazebo/gazebo.urdf.xacro" />
   <!-- materials for visualization -->
   <xacro:include filename="$(find youbot_description)/urdf/materials.urdf.xacro" />
@@ -29,12 +23,7 @@
        is the world frame). For more, see http://www.ros.org/wiki/xacro -->
 <!-- foot for arm-->
-  <xacro:youbot_base name="base" />
-  <xacro:youbot_plate name="plate" parent="base_link">
-    <origin xyz="-0.159 0 0.046" rpy="0 0 0" />
-  </xacro:youbot_plate>
-  <xacro:youbot_arm name="arm" parent="base_link">
-    <origin xyz="0.143 0 0.046" rpy="0 0 0" />
-  </xacro:youbot_arm>
-  <xacro:youbot_gripper name="gripper" parent="arm_link_5">
+  <link name="base_link">
+  </link>
+  <xacro:youbot_gripper name="gripper" parent="base_link">
     <origin xyz="0 0 0" rpy="0 0 0" />
   </xacro:youbot_gripper>

File: urdf/common.xacro (robot description, xacro)
@@ -1,9 +1,10 @@
 <?xml version="1.0"?>
-<robot>
-	<property name="M_PI" value="3.1415926535897931" />
+<robot
+    xmlns:xacro="http://www.ros.org/wiki/xacro">
+	<xacro:property name="M_PI" value="3.1415926535897931" />
 	<!-- Casters -->
-	<property name="cal_caster_fl" value="0.0" />
-	<property name="cal_caster_fr" value="0.0" />
-	<property name="cal_caster_bl" value="0.0" />
-	<property name="cal_caster_br" value="0.0" />
+	<xacro:property name="cal_caster_fl" value="0.0" />
+	<xacro:property name="cal_caster_fr" value="0.0" />
+	<xacro:property name="cal_caster_bl" value="0.0" />
+	<xacro:property name="cal_caster_br" value="0.0" />
 </robot>

File: urdf/youbot_arm/arm.gazebo.xacro (robot description, xacro)
@@ -3,5 +3,5 @@
        xmlns:controller="http://playerstage.sourceforge.net/gazebo/xmlschema/#controller"
        xmlns:interface="http://playerstage.sourceforge.net/gazebo/xmlschema/#interface"
-       xmlns:xacro="http://ros.org/wiki/xacro">
+       xmlns:xacro="http://www.ros.org/wiki/xacro">
 	<xacro:macro name="youbot_arm_gazebo" params="name">
 		<gazebo reference="${name}_link_0">

File: urdf/youbot_arm/arm.transmission.xacro (robot description, xacro)
@@ -3,5 +3,5 @@
        xmlns:controller="http://playerstage.sourceforge.net/gazebo/xmlschema/#controller"
        xmlns:interface="http://playerstage.sourceforge.net/gazebo/xmlschema/#interface"
-       xmlns:xacro="http://ros.org/wiki/xacro">
+       xmlns:xacro="http://www.ros.org/wiki/xacro">
 	<!-- reduction ratio doesn't affect the model-->
 	<!-- reduction ratio must not to be 0-->

File: urdf/youbot_arm/limits.urdf.xacro (robot description, xacro)
@@ -1,4 +1,4 @@
 <?xml version="1.0"?>
-<robot xmlns:xacro="http://ros.org/wiki/xacro">>
+<robot xmlns:xacro="http://www.ros.org/wiki/xacro">>
 	<!-- common properties -->
 	<xacro:property name="M_PI" value="3.1415926535897931" />

File: urdf/youbot_arm/view_arm.urdf.xacro (robot description, xacro)
@@ -3,15 +3,18 @@
         xmlns:controller="http://playerstage.sourceforge.net/gazebo/xmlschema/#controller"
         xmlns:interface="http://playerstage.sourceforge.net/gazebo/xmlschema/#interface"
-        xmlns:xacro="http://www.ros.org/wiki/xacro" >
+        xmlns:xacro="http://ros.org/wiki/xacro"
+	name="youbot_arm">
+    <xacro:include filename="$(find youbot_description)/urdf/youbot_gripper/gripper.urdf.xacro" />
 	<xacro:include filename="$(find youbot_description)/urdf/youbot_arm/arm.gazebo.xacro" />
 	<xacro:include filename="$(find youbot_description)/urdf/youbot_arm/arm.transmission.xacro" />
         <xacro:include filename="$(find youbot_description)/urdf/youbot_arm/limits.urdf.xacro" />
-	<xacro:macro name="youbot_arm" params="parent name *origin">
+	<property name="name" value="arm" />
+	<!--xacro:macro name="youbot_arm" params="parent name *origin"-->
 		<!-- joint between base_link and arm_0_link -->
-		<joint name="${name}_joint_0" type="fixed" >
+		<!--joint name="${name}_joint_0" type="fixed" >
 			<xacro:insert_block name="origin" />
 			<parent link="${parent}" />
 			<child link="${name}_link_0" />
-		</joint>
+		</joint-->
 		<link name="${name}_link_0">
 			<inertial>
@@ -119,5 +122,5 @@
 		</joint>-->
 		<joint name="${name}_joint_3" type="revolute">
-			<origin xyz="0.000 0.000 0.155" rpy="0 ${146 * M_PI / 180} 0"/>home/macs/catkin_ws/src/youbot_description/urdf/youbot_arm/arm.gazebo.xacr
+			<origin xyz="0.000 0.000 0.155" rpy="0 ${146 * M_PI / 180} 0"/>
 			<parent link="${name}_link_2"/>
 			<child link="${name}_link_3"/>
@@ -211,7 +214,10 @@
 			</collision>
 		</link>
+        <xacro:youbot_gripper parent="${name}_link_5" name="gripper">
+            <origin xyz="0 0 0" rpy="0 0 0"/>
+        </xacro:youbot_gripper>
 		<!-- extensions -->
 		<xacro:youbot_arm_gazebo name="${name}" />
 		<xacro:youbot_arm_transmission name="${name}" />
-	</xacro:macro>
+	<!--/xacro:macro-->
 </robot>

File: urdf/youbot_arm/view_arm1.urdf.xacro (robot description, xacro)
@@ -3,15 +3,18 @@
         xmlns:controller="http://playerstage.sourceforge.net/gazebo/xmlschema/#controller"
         xmlns:interface="http://playerstage.sourceforge.net/gazebo/xmlschema/#interface"
-        xmlns:xacro="http://www.ros.org/wiki/xacro" >
+        xmlns:xacro="http://ros.org/wiki/xacro"
+	name="youbot_arm">
+    <xacro:include filename="$(find youbot_description)/urdf/youbot_gripper/gripper.urdf.xacro" />
 	<xacro:include filename="$(find youbot_description)/urdf/youbot_arm/arm.gazebo.xacro" />
 	<xacro:include filename="$(find youbot_description)/urdf/youbot_arm/arm.transmission.xacro" />
         <xacro:include filename="$(find youbot_description)/urdf/youbot_arm/limits.urdf.xacro" />
-	<xacro:macro name="youbot_arm" params="parent name *origin">
+	<property name="name" value="arm_fake" />
+	<!--xacro:macro name="youbot_arm" params="parent name *origin"-->
 		<!-- joint between base_link and arm_0_link -->
-		<joint name="${name}_joint_0" type="fixed" >
+		<!--joint name="${name}_joint_0" type="fixed" >
 			<xacro:insert_block name="origin" />
 			<parent link="${parent}" />
 			<child link="${name}_link_0" />
-		</joint>
+		</joint-->
 		<link name="${name}_link_0">
 			<inertial>
@@ -119,5 +122,5 @@
 		</joint>-->
 		<joint name="${name}_joint_3" type="revolute">
-			<origin xyz="0.000 0.000 0.155" rpy="0 ${146 * M_PI / 180} 0"/>home/macs/catkin_ws/src/youbot_description/urdf/youbot_arm/arm.gazebo.xacr
+			<origin xyz="0.000 0.000 0.155" rpy="0 ${146 * M_PI / 180} 0"/>
 			<parent link="${name}_link_2"/>
 			<child link="${name}_link_3"/>
@@ -211,7 +214,10 @@
 			</collision>
 		</link>
+        <xacro:youbot_gripper parent="${name}_link_5" name="gripper_fake">
+            <origin xyz="0 0 0" rpy="0 0 0"/>
+        </xacro:youbot_gripper>
 		<!-- extensions -->
 		<xacro:youbot_arm_gazebo name="${name}" />
 		<xacro:youbot_arm_transmission name="${name}" />
-	</xacro:macro>
+	<!--/xacro:macro-->
 </robot>

File: urdf/youbot_base/base.gazebo.xacro (robot description, xacro)
@@ -3,5 +3,5 @@
        xmlns:controller="http://playerstage.sourceforge.net/gazebo/xmlschema/#controller"
        xmlns:interface="http://playerstage.sourceforge.net/gazebo/xmlschema/#interface"
-       xmlns:xacro="http://ros.org/wiki/xacro">
+       xmlns:xacro="http://www.ros.org/wiki/xacro">
   <xacro:macro name="youbot_base_gazebo">
     <gazebo reference="youbot_base">

File: urdf/youbot_base/base.transmission.xacro (robot description, xacro)
@@ -3,8 +3,8 @@
        xmlns:controller="http://playerstage.sourceforge.net/gazebo/xmlschema/#controller"
        xmlns:interface="http://playerstage.sourceforge.net/gazebo/xmlschema/#interface"
-       xmlns:xacro="http://ros.org/wiki/xacro">
-	<property name="wheel_mechanical_reduction" value="${624/35 * 80/18}" />
-	<property name="caster_mechanical_reduction" value="${624/35 * 80/18}" />
-	<property name="" value="0.360" />
+       xmlns:xacro="http://www.ros.org/wiki/xacro">
+	<xacro:property name="wheel_mechanical_reduction" value="${624/35 * 80/18}" />
+	<xacro:property name="caster_mechanical_reduction" value="${624/35 * 80/18}" />
+	<xacro:property name="" value="0.360" />
 	<xacro:macro name="youbot_base_transmission">
 		<!-- front left wheel -->

File: urdf/youbot_base/base.urdf.xacro (robot description, xacro)
@@ -3,33 +3,33 @@
        xmlns:controller="http://playerstage.sourceforge.net/gazebo/xmlschema/#controller"
        xmlns:interface="http://playerstage.sourceforge.net/gazebo/xmlschema/#interface"
-       xmlns:xacro="http://ros.org/wiki/xacro">
+       xmlns:xacro="http://www.ros.org/wiki/xacro" >
   <!-- sensors -->
   <xacro:include filename="$(find youbot_description)/urdf/youbot_base/base.gazebo.xacro"/>
   <xacro:include filename="$(find youbot_description)/urdf/youbot_base/base.transmission.xacro"/>
   <!-- simplified box collision geometry for base -->
-  <property name="base_size_x" value="0.570"/>
-  <property name="base_size_y" value="0.360"/>
-  <property name="base_size_z" value="0.100"/>
-  <property name="base_mass" value="22.0"/>
-  <property name="caster_offset_x" value="0.228"/>
-  <property name="caster_offset_y" value="0.158"/>
-  <property name="caster_offset_z" value="-0.034"/>
-  <property name="caster_mass" value="0.1"/>
-  <property name="wheel_offset_x" value="0.0"/>
-  <property name="wheel_offset_y" value="0.0"/>
-  <property name="wheel_offset_z" value="0.0"/>
-  <property name="wheel_mass" value="0.4"/>
-  <property name="wheel_radius" value="0.05"/>
-  <property name="wheel_length" value="0.005"/>
-  <property name="caster_joint_damping" value="1.0"/>
-  <property name="caster_joint_friction" value="1.0"/>
-  <property name="caster_joint_effort" value="30"/>
-  <property name="caster_joint_velocity" value="10"/>
-  <property name="caster_joint_safety_k_velocity" value="10.0"/>
-  <property name="wheel_joint_damping" value="1.0"/>
-  <property name="wheel_joint_friction" value="1.0"/>
-  <property name="wheel_joint_effort" value="30"/>
-  <property name="wheel_joint_velocity" value="10"/>
-  <property name="wheel_joint_safety_k_velocity" value="10.0"/>
+  <xacro:property name="base_size_x" value="0.570"/>
+  <xacro:property name="base_size_y" value="0.360"/>
+  <xacro:property name="base_size_z" value="0.100"/>
+  <xacro:property name="base_mass" value="22.0"/>
+  <xacro:property name="caster_offset_x" value="0.228"/>
+  <xacro:property name="caster_offset_y" value="0.158"/>
+  <xacro:property name="caster_offset_z" value="-0.034"/>
+  <xacro:property name="caster_mass" value="0.1"/>
+  <xacro:property name="wheel_offset_x" value="0.0"/>
+  <xacro:property name="wheel_offset_y" value="0.0"/>
+  <xacro:property name="wheel_offset_z" value="0.0"/>
+  <xacro:property name="wheel_mass" value="0.4"/>
+  <xacro:property name="wheel_radius" value="0.05"/>
+  <xacro:property name="wheel_length" value="0.005"/>
+  <xacro:property name="caster_joint_damping" value="1.0"/>
+  <xacro:property name="caster_joint_friction" value="1.0"/>
+  <xacro:property name="caster_joint_effort" value="30"/>
+  <xacro:property name="caster_joint_velocity" value="10"/>
+  <xacro:property name="caster_joint_safety_k_velocity" value="10.0"/>
+  <xacro:property name="wheel_joint_damping" value="1.0"/>
+  <xacro:property name="wheel_joint_friction" value="1.0"/>
+  <xacro:property name="wheel_joint_effort" value="30"/>
+  <xacro:property name="wheel_joint_velocity" value="10"/>
+  <xacro:property name="wheel_joint_safety_k_velocity" value="10.0"/>
   <xacro:macro name="youbot_base" params="name">
     <link name="${name}_footprint">

File: urdf/youbot_gripper/gripper.gazebo.xacro (robot description, xacro)
@@ -3,5 +3,5 @@
        xmlns:controller="http://playerstage.sourceforge.net/gazebo/xmlschema/#controller"
        xmlns:interface="http://playerstage.sourceforge.net/gazebo/xmlschema/#interface"
-       xmlns:xacro="http://ros.org/wiki/xacro">
+       xmlns:xacro="http://www.ros.org/wiki/xacro">
 	<xacro:macro name="youbot_gripper_gazebo" params="name">
 		<gazebo reference="${name}_palm_link">

File: urdf/youbot_gripper/gripper.transmission.xacro (robot description, xacro)
@@ -3,5 +3,5 @@
        xmlns:controller="http://playerstage.sourceforge.net/gazebo/xmlschema/#controller"
        xmlns:interface="http://playerstage.sourceforge.net/gazebo/xmlschema/#interface"
-       xmlns:xacro="http://ros.org/wiki/xacro">
+       xmlns:xacro="http://www.ros.org/wiki/xacro">
 	<xacro:macro name="youbot_gripper_transmission" params="name">
 		<transmission name="${name}_finger_l_trans">

File: urdf/youbot_gripper/gripper.urdf.xacro (robot description, xacro)
@@ -3,5 +3,5 @@
        xmlns:controller="http://playerstage.sourceforge.net/gazebo/xmlschema/#controller"
        xmlns:interface="http://playerstage.sourceforge.net/gazebo/xmlschema/#interface"
-       xmlns:xacro="http://ros.org/wiki/xacro">
+       xmlns:xacro="http://www.ros.org/wiki/xacro">
 	<xacro:include filename="$(find youbot_description)/urdf/youbot_gripper/gripper.gazebo.xacro" />
 	<xacro:include filename="$(find youbot_description)/urdf/youbot_gripper/gripper.transmission.xacro" />
@@ -10,5 +10,5 @@
 		<!-- joint between arm_7_link and sdh_palm_link -->
 		<joint name="${name}_palm_joint" type="fixed" >
-			<insert_block name="origin" />
+			<xacro:insert_block name="origin" />
 			<parent link="${parent}" />
 			<child link="${name}_palm_link" />
