Commit message: support for arm simulation and feedback visualization

File: urdf/youbot_gripper/limits.urdf.xacro (robot description, xacro)
@@ -1,9 +1,10 @@
 <?xml version="1.0"?>
-<robot>
+<robot
+    xmlns:xacro="http://www.ros.org/wiki/xacro">
 	<!-- common properties -->
-	<property name="M_PI" value="3.1415926535897931" />
-        <property name="threshold" value="0.001" />
+	<xacro:property name="M_PI" value="3.1415926535897931" />
+        <xacro:property name="threshold" value="0.001" />
 	<!-- fingers limits, values are in meters -->
-	<property name="finger_joint" value="${0.023 / 2.0}" />
-	<property name="finger_joint_soft" value="${(0.023 - threshold) / 2.0}" />
+	<xacro:property name="finger_joint" value="${0.023 / 2.0}" />
+	<xacro:property name="finger_joint_soft" value="${(0.023 - threshold) / 2.0}" />
 </robot>

File: urdf/youbot_plate/plate.urdf.xacro (robot description, xacro)
@@ -3,9 +3,9 @@
        xmlns:controller="http://playerstage.sourceforge.net/gazebo/xmlschema/#controller"
        xmlns:interface="http://playerstage.sourceforge.net/gazebo/xmlschema/#interface"
-       xmlns:xacro="http://ros.org/wiki/xacro">
+       xmlns:xacro="http://www.ros.org/wiki/xacro">
 	<xacro:macro name="youbot_plate" params="parent name *origin">
 		<!-- joint between arm_7_link and sdh_palm_link -->
 		<joint name="${name}_joint" type="fixed" >
-			<insert_block name="origin" />
+			<xacro:insert_block name="origin" />
 			<parent link="${parent}" />
 			<child link="${name}_link" />
